File: Schematics/Polyhymnia/MIDI_In.kicad_sch (KiCad schematic)
At the start: 5 parts, among them J1 DIN-5, U7 6N138

Commit message: Added audio amplifier schematics
Other:
- title: (none) -> MIDI-Input Unit
Changed lines of the file:
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@@
 	(generator "eeschema")
 	(generator_version "10.0")
-	(paper "A4")
+	(paper "A5")
+	(title_block
+		(title "MIDI-Input Unit")
+		(date "2026-06-13")
+		(rev "0.1")
+	)
 	(text_box "Note to myself:\nP2 = RCX\nP3 = Daten\nP4 3.3 V\nP5 = 5V"
 		(exclude_from_sim no)
