File: Schematics/Polyhymnia/Polyhymnia.kicad_sch (KiCad schematic)
At the start: 1 part, among them U1 Teensy4.1

Commit message: Squashed commit of the following:
commit 40d7620dede4bb8ae58b57caf8fc795e2b026afb
Author: Sebastian Murschall <sebastian.murschall@gmail.com>
Date:   Sun Jun 21 15:12:57 2026 +0200

    Update README.org

commit 70c3d47f3131ce146337862403d6c48c4c7a9d9c
Author: Sebastian Murschall <sebastian.murschall@gmail.com>
Date:   Sun Jun 21 15:08:39 2026 +0200

    updated schematics

commit e9316d961a51c20d4760f1c1fbe43982f1e61518
Author: Sebastian Murschall <sebastian.murschall@gmail.com>
Date:   Sun Jun 21 15:08:24 2026 +0200

    Added first draft for an enclosure
Parts:
- added R55: 50, symbol Device:R
- added U11: CR2013-MI2120, Display:CR2013-MI2120, symbol Driver_Display:CR2013-MI2120
Connections:
- net AudioShield_DOUT is gone; now on net AudioShield_MEMCS: U1.8 (6_OUT1D)
- net +3V3: now also U11.1 (VCC)
- net AudioShield_BCLK: now also U1.43 (21_A7_RX5_BCLK1); no longer U1.21 (29_TX7)
- net AudioShield_DIN: now also U1.10 (8_TX2_IN1), U1.9 (7_RX2_OUT1A); no longer U1.7 (5_IN2)
- net AudioShield_LRCLK: now also U1.42 (20_A6_TX5_LRCLK1); no longer U1.20 (28_RX7)
- net AudioShield_MCLK: now also U1.45 (23_A9_CRX1_MCLK1); no longer U1.23 (31_CTX3)
- net AudioShield_MEMCS: no longer U1.6 (4_BCLK2)
- net AudioShield_MISO: now also U1.14 (12_MISO_MQSL); no longer U1.12 (10_CS_MQSR)
- net AudioShield_MOSI: now also U1.13 (11_MOSI_CTX1); no longer U1.11 (9_OUT1C)
- net AudioShield_SCK: now also U1.35 (13_SCK_LED); no longer U1.13 (11_MOSI_CTX1)
- net AudioShield_SCL: now also U1.41 (19_A5_SCL); no longer U1.19 (27_A13_SCK1)
- net AudioShield_SDA: now also U1.40 (18_A4_SDA); no longer U1.18 (26_A12_MOSI1)
- net AudioShield_SDCS: now also U1.12 (10_CS_MQSR); no longer U1.10 (8_TX2_IN1)
- net Encoder Multiplexer/SS: no longer U1.28 (36_CS)
- net GND: now also U1.1 (GND), U11.2 (GND)
- net MIDI_In/MIDI_IN: now also U11.5 (D/~{C})
- net at U1.3 (1_TX1_CTX2_MISO1): now also U11.9 (MISO)
- new net: R55.1, U11.8 (LED)
- new net: R55.2, U1.20 (28_RX7)
- new net: U1.21 (29_TX7), U11.4 (RESET)
- new net: U1.18 (26_A12_MOSI1), U11.6 (MOSI)
- new net: U1.19 (27_A13_SCK1), U11.7 (SCK)
