File: Schematics/Polyhymnia/osc_unit.kicad_sch (KiCad schematic)
At the start: 7 parts, among them J4 Conn_02x05_Counter_Clockwise, SW10 RotaryEncoder, SW5 RotaryEncoder

Commit message: Merge
Parts:
- added R33, R36, R39, R42: 68 Ohm, symbol Device:R
- renumbered D35 to D34, D37 to D35, D34 to D37, SW10 to SW1, SW5 to SW2
Connections:
- net LED_SAW: now also R36.1; no longer J4.2 (Pin_2)
- net LED_SINE: now also R33.1; no longer J4.7 (Pin_7)
- net LED_SQUARE: now also R42.1; no longer J4.6 (Pin_6)
- net LED_TRIANGLE: now also R39.1; no longer J4.3 (Pin_3)
- new net: J4.2 (Pin_2), R36.2
- new net: J4.7 (Pin_7), R33.2
- new net: J4.3 (Pin_3), R39.2
- new net: J4.6 (Pin_6), R42.2
Other:
- note added: "Note to myself: 04 Frequency PhaseA PC0 05 Frequency PhaseB PC1 06 LED PC2 07 LED PC3 08 LED PC4 09 LED DEAD 10 A PC6 10 GND 11 B PC7"
- title: (none) -> Oscillator Control Unit
